File: m.2_usd.kicad_pcb (KiCad board)
At the start: 4 copper layers, 22 x 26 mm, 5 parts, among them J1 Bus_M.2_Socket_E, J2 112C-TBAR-R02

Commit message: Added extensive via stitching
Parts:
- removed REF**: m2-outer2230, footprints:m2-outer2230
- J1: footprint footprints:m2-padKeyE -> footprints:m2-padKeyE-2230
Routing:
- net GND: track 88.3 -> 90.5 mm, vias 31 -> 55
- net DAT3: track 22.2 -> 20.6 mm
Other:
- board size 22 x 26 mm -> 22 x 30 mm

Commit message: ERC and DRC pass
Routing:
- net +3V3: track 45.0 -> 56.8 mm
- net GND: vias 55 -> 56
Other:
- board text added: "M.M. 2024 M.2 to micro SD adapter"
Changed lines of the file:
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@@
       (outputformat 1)
       (mirror false)
-      (drillshape 1)
+      (drillshape 0)
       (scaleselection 1)
-      (outputdirectory "")
+      (outputdirectory "gerbers")
     )
   )
@@
         (effects (font (size 0.8 0.8) (thickness 0.15)))
     )
-    (fp_line (start -11 -4) (end 11 -4)
+    (fp_line (start -10 -4) (end 10 -4)
       (stroke (width 0.01) (type solid)) (layer "F.SilkS"))
     (fp_line (start 0 0) (end 0 -30)
@@
     (property "ki_keywords" "112C-TBAR-R02")
     (attr smd)
-    (fp_text reference "J2" (at 0 -2.1509 -90 unlocked) (layer "F.SilkS")
+    (fp_text reference "J2" (at -6.25 -8.3 -90 unlocked) (layer "F.SilkS")
         (effects (font (size 1 1) (thickness 0.15)))
     )
@@
     (property "ki_keywords" "cap capacitor")
     (attr smd)
-    (fp_text reference "C1" (at 0 1.43 90) (layer "B.SilkS")
+    (fp_text reference "C1" (at 2.85 -0.11 90) (layer "B.SilkS")
         (effects (font (size 1 1) (thickness 0.15)) (justify mirror))
     )
@@
     (property "ki_keywords" "cap capacitor")
     (attr smd)
-    (fp_text reference "C2" (at 0 1.43 90) (layer "B.SilkS")
+    (fp_text reference "C2" (at 2.65 -0.05 90) (layer "B.SilkS")
         (effects (font (size 1 1) (thickness 0.15)) (justify mirror))
     )
@@
       (rotate (xyz 0 0 0))
     )
+  )
+  (gr_text "M.M. 2024\nM.2 to micro SD adapter" (at 10.05 -28.65 90) (layer "B.SilkS")
+    (effects (font (size 1 1) (thickness 0.1)) (justify left bottom mirror))
+  )
+  (gr_text "M.M. 2024\nM.2 to micro SD adapter" (at 10.15 -28.9 90) (layer "F.SilkS")
+    (effects (font (size 1 1) (thickness 0.1)) (justify right bottom))
   )
   (segment (start -9.25 -2.9) (end -9.25 -1.55) (width 0.35) (layer "F.Cu") (net 1))
@@
   (via (at 6.95 -15.8) (size 0.6) (drill 0.3) (layers "F.Cu" "B.Cu") (free) (net 1))
   (via (at -2.5 -15.8) (size 0.6) (drill 0.3) (layers "F.Cu" "B.Cu") (free) (net 1))
+  (via (at 3.575 -7.925) (size 0.6) (drill 0.3) (layers "F.Cu" "B.Cu") (free) (net 1))
   (via (at -1.9 -9.5) (size 0.6) (drill 0.3) (layers "F.Cu" "B.Cu") (free) (net 1))
   (via (at 7.15 -14.35) (size 0.6) (drill 0.3) (layers "F.Cu" "B.Cu") (free) (net 1))
@@
   (segment (start -1.2491 -14.8) (end -4.675 -14.8) (width 0.342392) (layer "F.Cu") (net 2))
   (via (at -5 -14.475) (size 0.6) (drill 0.3) (layers "F.Cu" "B.Cu") (net 2))
-  (segment (start -7.625 -14.475) (end -6.21 -14.475) (width 0.342392) (layer "B.Cu") (net 2))
+  (segment (start -9 -13) (end -7.525 -14.475) (width 0.35) (layer "B.Cu") (net 2))
+  (segment (start -7.525 -14.475) (end -6.21 -14.475) (width 0.35) (layer "B.Cu") (net 2))
+  (segment (start -9 -1.55) (end -8.5 -1.55) (width 0.35) (layer "B.Cu") (net 2))
   (segment (start -3.7 -19.5) (end -3.7 -14.475) (width 0.342392) (layer "B.Cu") (net 2))
   (segment (start -3.2 -20) (end -3.7 -19.5) (width 0.342392) (layer "B.Cu") (net 2))
+  (segment (start -9 -1.55) (end -9 -13) (width 0.35) (layer "B.Cu") (net 2))
   (segment (start 9 -3.1) (end 9 -16.685786) (width 0.342392) (layer "B.Cu") (net 2))
   (segment (start 8.707107 -17.392893) (end 6.1 -20) (width 0.342392) (layer "B.Cu") (net 2))
@@
   (segment (start 9 -1.55) (end 9 -3.1) (width 0.342392) (layer "B.Cu") (net 2))
   (segment (start 6.1 -20) (end -3.2 -20) (width 0.342392) (layer "B.Cu") (net 2))
-  (segment (start 9 -3.1) (end 8.9 -3.2) (width 0.342392) (layer "B.Cu") (net 2))
-  (segment (start -9 -13.1) (end -7.625 -14.475) (width 0.342392) (layer "B.Cu") (net 2))
   (segment (start 9 -1.55) (end 8.546196 -1.55) (width 0.342392) (layer "B.Cu") (net 2))
   (segment (start -5 -14.475) (end -6.21 -14.475) (width 0.342392) (layer "B.Cu") (net 2))
@@
   (segment (start 4.315775 -16.184225) (end 4.315775 -4.772136) (width 0.342392) (layer "B.Cu") (net 16))
   (segment (start 4.25 -16.25) (end 4.315775 -16.184225) (width 0.342392) (layer "B.Cu") (net 16))
+  (zone (net 0) (net_name "") (layer "F.Cu") (hatch edge 0.5)
+    (connect_pads (clearance 0))
+    (min_thickness 0.0889) (filled_areas_thickness no)
+    (keepout (tracks allowed) (vias allowed) (pads allowed) (copperpour not_allowed) (footprints allowed))
+    (fill (thermal_gap 0.5) (thermal_bridge_width 0.5))
+    (polygon
+      (pts
+        (arc (start -4.25 -30) (mid 0 -25.75) (end 4.25 -30))
+        (arc (start 2.75 -30) (mid 0 -27.25) (end -2.75 -30))
+      )
+    )
+  )
   (zone (net 1) (net_name "GND") (layers "F.Cu" "In1.Cu" "In2.Cu" "B.Cu") (hatch edge 0.5)
     (connect_pads (clearance 0.0889))
