File: m.2_usd.kicad_sch (KiCad schematic)
At the start: 4 parts, among them J1 Bus_M.2_Socket_E, J2 112C-TBAR-R02

Commit message: Added extensive via stitching
Parts:
- J1: footprint footprints:m2-padKeyE -> footprints:m2-padKeyE-2230
- J2: footprint 112C-TBAR-R02_ATT -> footprints:112C-TBAR-R02_ATT
Changed lines of the file:
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@@
       (effects (font (size 1.27 1.27)) (justify left))
     )
-    (property "Footprint" "footprints:m2-padKeyE" (at 110.49 95.25 0)
+    (property "Footprint" "footprints:m2-padKeyE-2230" (at 110.49 95.25 0)
       (effects (font (size 1.27 1.27)) hide)
     )
@@
       (effects (font (size 1.524 1.524)))
     )
-    (property "Footprint" "112C-TBAR-R02_ATT" (at 205.74 99.06 0)
+    (property "Footprint" "footprints:112C-TBAR-R02_ATT" (at 205.74 99.06 0)
       (effects (font (size 1.27 1.27) italic) hide)
     )

Commit message: ERC and DRC pass
Connections:
- no-connect marks 15 -> 46
Changed lines of the file:
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@@
   )
   (no_connect (at 85.09 93.98))
+  (no_connect (at 135.89 127))
+  (no_connect (at 135.89 157.48))
   (no_connect (at 85.09 88.9))
+  (no_connect (at 85.09 119.38))
+  (no_connect (at 85.09 129.54))
+  (no_connect (at 85.09 160.02))
   (no_connect (at 85.09 99.06))
   (no_connect (at 85.09 86.36))
@@
   (no_connect (at 135.89 111.76))
   (no_connect (at 85.09 96.52))
+  (no_connect (at 135.89 93.98))
+  (no_connect (at 135.89 106.68))
+  (no_connect (at 135.89 99.06))
+  (no_connect (at 85.09 132.08))
+  (no_connect (at 85.09 121.92))
+  (no_connect (at 135.89 165.1))
+  (no_connect (at 135.89 149.86))
+  (no_connect (at 135.89 91.44))
   (no_connect (at 85.09 83.82))
+  (no_connect (at 85.09 134.62))
   (no_connect (at 85.09 104.14))
+  (no_connect (at 135.89 96.52))
+  (no_connect (at 85.09 127))
   (no_connect (at 135.89 81.28))
   (no_connect (at 85.09 78.74))
+  (no_connect (at 85.09 114.3))
   (no_connect (at 85.09 106.68))
+  (no_connect (at 135.89 129.54))
+  (no_connect (at 85.09 157.48))
+  (no_connect (at 85.09 142.24))
+  (no_connect (at 85.09 149.86))
+  (no_connect (at 135.89 101.6))
+  (no_connect (at 135.89 152.4))
+  (no_connect (at 135.89 160.02))
+  (no_connect (at 135.89 162.56))
+  (no_connect (at 135.89 124.46))
+  (no_connect (at 85.09 144.78))
   (no_connect (at 135.89 78.74))
+  (no_connect (at 85.09 154.94))
+  (no_connect (at 85.09 137.16))
+  (no_connect (at 85.09 116.84))
   (no_connect (at 135.89 114.3))
+  (no_connect (at 135.89 104.14))
   (no_connect (at 135.89 88.9))
   (wire (pts (xy 139.7 139.7) (xy 135.89 139.7))
     (stroke (width 0) (type default))
   )
-  (wire (pts (xy 140.97 137.16) (xy 135.89 137.16))
+  (wire (pts (xy 139.7 137.16) (xy 135.89 137.16))
     (stroke (width 0) (type default))
   )
@@
     (stroke (width 0) (type default))
   )
-  (global_label "CMD" (shape output) (at 140.97 137.16 0) (fields_autoplaced)
+  (global_label "CMD" (shape bidirectional) (at 139.7 137.16 0) (fields_autoplaced)
     (effects (font (size 1.27 1.27)) (justify left))
-    (property "Intersheetrefs" "${INTERSHEET_REFS}" (at 147.9466 137.16 0)
+    (property "Intersheetrefs" "${INTERSHEET_REFS}" (at 147.7879 137.16 0)
       (effects (font (size 1.27 1.27)) (justify left) hide)
     )
@@
     )
   )
-  (global_label "CMD" (shape input) (at 200.66 104.14 180) (fields_autoplaced)
+  (global_label "CMD" (shape bidirectional) (at 200.66 104.14 180) (fields_autoplaced)
     (effects (font (size 1.27 1.27)) (justify right))
-    (property "Intersheetrefs" "${INTERSHEET_REFS}" (at 193.6834 104.14 0)
+    (property "Intersheetrefs" "${INTERSHEET_REFS}" (at 192.5721 104.14 0)
       (effects (font (size 1.27 1.27)) (justify right) hide)
     )
